File: pcbs/switch_plate/switch_plate.kicad_pcb (KiCad board)
At the start: 2 copper layers, 94 x 70.7 mm, 4 parts

Commit message: feat: moving the pinky column downward, adding backplate
Other:
- outline, holes or cut-outs redrawn
Changed lines of the file:
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@@
       (drillshape 0)
       (scaleselection 1)
-      (outputdirectory "./gerbers/")
+      (outputdirectory "../../gerbers/top_plate/")
     )
   )
@@
   (gr_line (start 162.5 110.7) (end 162.5 96.7)
     (stroke (width 0.15) (type default)) (layer "Edge.Cuts"))
-  (gr_line (start 108.5 76.7) (end 108.5 62.7)
+  (gr_line (start 108.5 88.7) (end 108.5 74.7)
     (stroke (width 0.15) (type default)) (layer "Edge.Cuts"))
   (gr_line (start 180.5 127.7) (end 180.5 113.7)
@@
   (gr_line (start 104.5 129.2) (end 104.5 62.7)
     (stroke (width 0.15) (type default)) (layer "Edge.Cuts"))
-  (gr_line (start 108.5 79.7) (end 122.5 79.7)
+  (gr_line (start 108.5 91.7) (end 122.5 91.7)
     (stroke (width 0.15) (type default)) (layer "Edge.Cuts"))
   (gr_line (start 162.5 113.7) (end 176.5 113.7)
@@
   (gr_line (start 144.5 96.7) (end 158.5 96.7)
     (stroke (width 0.15) (type default)) (layer "Edge.Cuts"))
-  (gr_line (start 122.5 93.7) (end 108.5 93.7)
+  (gr_line (start 122.5 105.7) (end 108.5 105.7)
     (stroke (width 0.15) (type default)) (layer "Edge.Cuts"))
   (gr_line (start 180.5 79.7) (end 194.5 79.7)
@@
   (gr_line (start 180.5 93.7) (end 180.5 79.7)
     (stroke (width 0.15) (type default)) (layer "Edge.Cuts"))
-  (gr_line (start 122.5 110.7) (end 108.5 110.7)
+  (gr_line (start 122.5 122.7) (end 108.5 122.7)
     (stroke (width 0.15) (type default)) (layer "Edge.Cuts"))
-  (gr_line (start 108.5 93.7) (end 108.5 79.7)
+  (gr_line (start 108.5 105.7) (end 108.5 91.7)
     (stroke (width 0.15) (type default)) (layer "Edge.Cuts"))
   (gr_line (start 180.5 113.7) (end 194.5 113.7)
     (stroke (width 0.15) (type default)) (layer "Edge.Cuts"))
-  (gr_line (start 122.5 76.7) (end 108.5 76.7)
+  (gr_line (start 122.5 88.7) (end 108.5 88.7)
     (stroke (width 0.15) (type default)) (layer "Edge.Cuts"))
   (gr_line (start 158.5 93.7) (end 144.5 93.7)
@@
   (gr_line (start 162.5 76.7) (end 162.5 62.7)
     (stroke (width 0.15) (type default)) (layer "Edge.Cuts"))
-  (gr_line (start 122.5 62.7) (end 122.5 76.7)
+  (gr_line (start 122.5 74.7) (end 122.5 88.7)
     (stroke (width 0.15) (type default)) (layer "Edge.Cuts"))
   (gr_line (start 162.5 62.7) (end 176.5 62.7)
@@
   (gr_line (start 140.5 76.7) (end 126.5 76.7)
     (stroke (width 0.15) (type default)) (layer "Edge.Cuts"))
-  (gr_line (start 108.5 96.7) (end 122.5 96.7)
+  (gr_line (start 108.5 108.7) (end 122.5 108.7)
     (stroke (width 0.15) (type default)) (layer "Edge.Cuts"))
   (gr_line (start 194.5 93.7) (end 180.5 93.7)
@@
   (gr_arc (start 198.5 129.2) (mid 197.914214 130.614214) (end 196.5 131.2)
     (stroke (width 0.15) (type default)) (layer "Edge.Cuts"))
-  (gr_line (start 108.5 110.7) (end 108.5 96.7)
+  (gr_line (start 108.5 122.7) (end 108.5 108.7)
     (stroke (width 0.15) (type default)) (layer "Edge.Cuts"))
-  (gr_line (start 122.5 79.7) (end 122.5 93.7)
+  (gr_line (start 122.5 91.7) (end 122.5 105.7)
     (stroke (width 0.15) (type default)) (layer "Edge.Cuts"))
-  (gr_line (start 108.5 62.7) (end 122.5 62.7)
+  (gr_line (start 108.5 74.7) (end 122.5 74.7)
     (stroke (width 0.15) (type default)) (layer "Edge.Cuts"))
   (gr_line (start 140.5 110.7) (end 126.5 110.7)
     (stroke (width 0.15) (type default)) (layer "Edge.Cuts"))
-  (gr_line (start 122.5 96.7) (end 122.5 110.7)
+  (gr_line (start 122.5 108.7) (end 122.5 122.7)
     (stroke (width 0.15) (type default)) (layer "Edge.Cuts"))
   (gr_line (start 144.5 79.7) (end 158.5 79.7)
